File: kicad/classab-amp.kicad_sch (KiCad schematic)
At the start: 60 parts, among them J1 SPEAKER, J3 INPUT, Q1 BC547, Q10 MJL3218C, Q11 BD140, Q12 MJL1302C, Q13 BC547, Q14 BC557, Q2 BC547, Q3 BC557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

Commit message: Post 1.0 adjutments
Parts:
- added C6: 100n, symbol Device:C
Connections:
- net at C5.2, D6.2 (A), Q6.2 (C)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: now also C6.1
- net at D3.1 (K), Q11.3 (B), Q7.1 (E)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: now also C6.2
Changed lines of the file:
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@@
 	)
 	(junction
+		(at 176.53 118.11)
+		(diameter 0)
+		(color 0 0 0 0)
+	)
+	(junction
 		(at 115.57 29.21)
 		(diameter 0)
@@
 	(wire
 		(pts
+			(xy 176.53 115.57) (xy 176.53 118.11)
+		)
+		(stroke
+			(width 0)
+			(type default)
+		)
+	)
+	(wire
+		(pts
 			(xy 207.01 46.99) (xy 207.01 48.26)
 		)
@@
 	(wire
 		(pts
+			(xy 176.53 118.11) (xy 182.88 118.11)
+		)
+		(stroke
+			(width 0)
+			(type default)
+		)
+	)
+	(wire
+		(pts
 			(xy 154.94 118.11) (xy 168.91 118.11)
 		)
@@
 	(wire
 		(pts
-			(xy 168.91 118.11) (xy 182.88 118.11)
+			(xy 168.91 118.11) (xy 176.53 118.11)
 		)
 		(stroke
@@
 	(wire
 		(pts
+			(xy 176.53 107.95) (xy 176.53 90.17)
+		)
+		(stroke
+			(width 0)
+			(type default)
+		)
+	)
+	(wire
+		(pts
 			(xy 207.01 63.5) (xy 220.98 63.5)
 		)
@@
 	(wire
 		(pts
+			(xy 168.91 90.17) (xy 176.53 90.17)
+		)
+		(stroke
+			(width 0)
+			(type default)
+		)
+	)
+	(wire
+		(pts
 			(xy 220.98 99.06) (xy 220.98 101.6)
 		)
@@
 					(unit 1)
 				)
+			)
+		)
+	)
+	(symbol
+		(lib_id "Device:C")
+		(at 176.53 111.76 0)
+		(unit 1)
+		(exclude_from_sim no)
+		(in_bom yes)
+		(on_board yes)
+		(dnp no)
+		(fields_autoplaced yes)
+		(property "Reference" "C6"
+			(at 180.34 110.4899 0)
+			(effects
+				(font
+					(size 1.27 1.27)
+				)
+				(justify left)
+			)
+		)
+		(property "Value" "100n"
+			(at 180.34 113.0299 0)
+			(effects
+				(font
+					(size 1.27 1.27)
+				)
+				(justify left)
+			)
+		)
+		(property "Footprint" ""
+			(at 177.4952 115.57 0)
+			(effects
+				(font
+					(size 1.27 1.27)
+				)
+				(hide yes)
+			)
+		)
+		(property "Datasheet" "~"
+			(at 176.53 111.76 0)
+			(effects
+				(font
+					(size 1.27 1.27)
+				)
+				(hide yes)
+			)
+		)
+		(property "Description" "Unpolarized capacitor"
+			(at 176.53 111.76 0)
+			(effects
+				(font
+					(size 1.27 1.27)
+				)
+				(hide yes)
+			)
+		)
+		(pin "1"
+		)
+		(pin "2"
+		)
+		(instances
+			(project ""
+				(path "/856f1e14-388c-4d87-abe9-3c0c6310ec29"
+					(reference "C6")
+					(unit 1)
+				)

Commit message: Post build adjustments
Parts:
- added D10, D7, D8, D9: 1N5400, Diode_THT:D_DO-201AD_P15.24mm_Horizontal, symbol Diode:1N5400
- R10, R14: value 1k -> 150
- R12: value 6.8k -> 15k
Connections:
- net B+: now also D7.2 (A), D8.1 (K)
- net B-: now also D10.1 (K), D9.2 (A)
- net GND: now also D7.1 (K), D9.1 (K)
- net at Q10.3 (E), R16.1, R18.2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: now also D8.2 (A)
- net at Q12.3 (E), R17.2, R19.1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: now also D10.2 (A)
Other:
- moved on the sheet: C3, J1, L1, R20, R21
