File: kicad/classab-amp.kicad_pcb (KiCad board)
At the start: 2 copper layers, 46 parts, among them Q1 BC547, Q10 MJL3218C, Q11 MJE350C, Q12 MJL1302C, Q2 BC547, Q3 BC557, Q4 BC557, Q5 BC547, Q6 BC557, Q7 BC547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

Commit message: PCB layout
Parts:
- removed C7, C8: 4700u, Capacitor_THT:CP_Radial_D18.0mm_P7.50mm
- removed D7, D8, D9: 1N5400, Diode_THT:D_DO-201AD_P15.24mm_Horizontal
- removed R22: 100, Resistor_THT:R_Axial_DIN0204_L3.6mm_D1.6mm_P7.62mm_Horizontal
- added ?: , , F.Cu at (187.5, 129.5)
- added C11: 470p, Capacitor_THT:C_Rect_L7.2mm_W3.0mm_P5.00mm_FKS2_FKP2_MKS2_MKP2, F.Cu at (209.9, 73.2)
- added C12: 470p, Capacitor_THT:C_Rect_L7.2mm_W3.0mm_P5.00mm_FKS2_FKP2_MKS2_MKP2, F.Cu at (209.9, 93.5)
- added C13: 4700u, Capacitor_THT:CP_Radial_D18.0mm_P7.50mm, F.Cu at (228.1, 111.4)
- added C14: 4700u, Capacitor_THT:CP_Radial_D18.0mm_P7.50mm, F.Cu at (228.7, 44.2)
- added C15: 100n, Capacitor_THT:C_Rect_L7.2mm_W3.0mm_P5.00mm_FKS2_FKP2_MKS2_MKP2, F.Cu at (241.3, 121.4)
- added C16: 100n, Capacitor_THT:C_Rect_L7.2mm_W3.0mm_P5.00mm_FKS2_FKP2_MKS2_MKP2, F.Cu at (245.8, 42.2)
- added C2: 220p, Capacitor_THT:C_Rect_L7.2mm_W3.0mm_P5.00mm_FKS2_FKP2_MKS2_MKP2, F.Cu at (206.3, 100.8)
- added C5: 50p, Capacitor_THT:C_Rect_L7.2mm_W3.0mm_P5.00mm_FKS2_FKP2_MKS2_MKP2, F.Cu at (209.8, 63.2)
- added Q13: BC547, Package_TO_SOT_THT:TO-92_Inline, F.Cu at (217.0, 72.2)
- added Q14: BC557, Package_TO_SOT_THT:TO-92_Inline, F.Cu at (217.0, 91.9)
- added R17: 0.22, Resistor_THT:R_Axial_DIN0414_L11.9mm_D4.5mm_P15.24mm_Horizontal, F.Cu at (244.0, 83.8)
- added R20: 10, Resistor_THT:R_Axial_DIN0414_L11.9mm_D4.5mm_P15.24mm_Horizontal, F.Cu at (236.0, 83.8)
- added R21: 10, Resistor_THT:R_Axial_DIN0414_L11.9mm_D4.5mm_P15.24mm_Horizontal, F.Cu at (236.1, 63.7)
- added R24: 1k, Resistor_THT:R_Axial_DIN0204_L3.6mm_D1.6mm_P7.62mm_Horizontal, F.Cu at (223.1, 74.5)
- added R25: 8.2k, Resistor_THT:R_Axial_DIN0204_L3.6mm_D1.6mm_P7.62mm_Horizontal, F.Cu at (229.1, 74.7)
- added R26: 8.2k, Resistor_THT:R_Axial_DIN0204_L3.6mm_D1.6mm_P7.62mm_Horizontal, F.Cu at (229.1, 87.2)
- added R27: 1k, Resistor_THT:R_Axial_DIN0204_L3.6mm_D1.6mm_P7.62mm_Horizontal, F.Cu at (223.1, 94.7)
- added REF**: MountingHole_2.1mm, MountingHole:MountingHole_2.1mm, F.Cu at (268.0, 35.0)
- added REF**: MountingHole_2.1mm, MountingHole:MountingHole_2.1mm, F.Cu at (267.0, 129.5)
- added REF**: MountingHole_2.1mm, MountingHole:MountingHole_2.1mm, F.Cu at (188.5, 35.0)
- C3: value 100u -> 100n; footprint Capacitor_THT:CP_Radial_D4.0mm_P1.50mm -> Capacitor_THT:C_Rect_L7.2mm_W3.0mm_P5.00mm_FKS2_FKP2_MKS2_MKP2
- D3: value 1N4148 -> 1N4001; footprint Diode_THT:D_DO-35_SOD27_P7.62mm_Horizontal -> Diode_THT:D_DO-41_SOD81_P10.16mm_Horizontal
- D6: value 1N5400 -> 1N4001; footprint Diode_THT:D_DO-201AD_P15.24mm_Horizontal -> Diode_THT:D_DO-41_SOD81_P10.16mm_Horizontal
- Q11: value MJE350C -> BD140
- Q6: value BC557 -> BD140; footprint Package_TO_SOT_THT:TO-92_Inline -> Package_TO_SOT_THT:TO-126-3_Vertical
- Q7, Q8: value BC547 -> BD139; footprint Package_TO_SOT_THT:TO-92_Inline -> Package_TO_SOT_THT:TO-126-3_Vertical
- Q9: value MJ340C -> BD139
- R12: value 10k -> 6.8k
- R15: value 100 -> 10; footprint Resistor_THT:R_Axial_DIN0204_L3.6mm_D1.6mm_P7.62mm_Horizontal -> Resistor_THT:R_Axial_DIN0414_L11.9mm_D4.5mm_P15.24mm_Horizontal
- R16: footprint Resistor_THT:R_Axial_DIN0614_L14.3mm_D5.7mm_P25.40mm_Horizontal -> Resistor_THT:R_Axial_DIN0414_L11.9mm_D4.5mm_P15.24mm_Horizontal
- R8: value 100 -> 1k
- RV1: footprint Resistor_THT:R_Axial_DIN0204_L3.6mm_D1.6mm_P7.62mm_Horizontal -> footprints:TRIM_T93YA103KT20
- moved D6 134.4 mm to (239.3, 56.9), turned to 0 degrees
- moved R15 101.1 mm to (197.6, 124.1), turned to 90 degrees
- moved R16 78.3 mm to (244.0, 63.7), turned to -90 degrees
- moved D1 62.2 mm to (211.3, 124.2)
- moved C1 47.0 mm to (189.8, 110.2)
- moved R14 46.4 mm to (261.4, 85.5), turned to -90 degrees
- moved R1 46.2 mm to (194.3, 100.0), turned to 0 degrees
- moved Q5 45.5 mm to (209.0, 108.9)
- moved Q2 45.4 mm to (201.4, 93.5)
- moved Q1 45.3 mm to (190.2, 93.5)
- moved R5 45.2 mm to (216.2, 116.5)
- moved D2 44.4 mm to (206.2, 124.2)
- moved Q8 35.7 mm to (267.6, 85.0), turned to -90 degrees
- moved Q9 35.2 mm to (267.6, 62.9)
- moved R6 35.0 mm to (206.0, 112.7)
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Connections:
- C1 pad 1: unconnected-(C1-Pad1) -> INPUT
- D6 pad 1: B+ -> Net-(D6-K)
- D6 pad 2: AC2 -> Net-(D6-A)
- Q11 pad 3: Net-(Q11-B) -> Net-(D3-K)
- Q6 pad 1: Net-(D3-A) -> Net-(Q6-E)
- Q6 pad 2: Net-(Q6-B) -> Net-(D6-A)
- Q6 pad 3: Net-(Q6-E) -> Net-(Q6-B)
- Q7 pad 2: Net-(Q7-B) -> Net-(D6-A)
- Q7 pad 3: Net-(Q7-E) -> Net-(Q7-B)
- Q8 pad 1: Net-(Q7-E) -> Net-(Q8-E)
- Q8 pad 2: Net-(D4-A) -> Net-(D3-K)
- Q8 pad 3: Net-(Q8-E) -> Net-(D4-A)
- Q9 pad 3: Net-(Q9-B) -> Net-(D6-A)
- R11 pad 1: Net-(R11-Pad1) -> Net-(D6-A)
- R12 pad 1: Net-(Q7-B) -> Net-(R12-Pad1)
- R12 pad 2: Net-(Q7-E) -> Net-(D3-K)
- R13 pad 2: CT -> GND
- R15 pad 1: Net-(Q9-B) -> CHASSIS
- R15 pad 2: Net-(D3-A) -> GND
- R2 pad 2: CT -> GND
- R6 pad 2: CT -> GND
- R7 pad 1: CT -> GND
- R8 pad 1: Net-(Q1-C) -> Net-(Q6-B)
- R8 pad 2: Net-(Q6-B) -> Net-(Q1-C)
- RV1 pad 1: Net-(D3-A) -> Net-(Q7-B)
- RV1 pad 2: Net-(D3-A) -> Net-(Q7-B)
Routing:
- net Net-(D6-A): track 0.00 -> 99.5 mm
- net Net-(Q13-E): track 0.00 -> 86.8 mm
- net Net-(Q10-E): track 0.00 -> 81.1 mm
- net Net-(Q12-E): track 0.00 -> 68.5 mm
- net Net-(D6-K): track 0.00 -> 67.4 mm
- net Net-(D3-K): track 0.00 -> 61.6 mm
- net Net-(Q1-C): track 0.00 -> 61.5 mm
- net GND: track 0.00 -> 43.5 mm
- net Net-(D3-A): track 0.00 -> 41.7 mm
- net Net-(Q2-C): track 0.00 -> 39.5 mm
- net Net-(Q1-E): track 0.00 -> 34.4 mm
- net Net-(Q10-B): track 0.00 -> 32.0 mm
- net Net-(D4-A): track 0.00 -> 29.0 mm
- net B-: track 26.0 -> 0.00 mm
- net Net-(Q11-E): track 0.00 -> 25.2 mm
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- added copper zone on B.Cu, net B+
- added copper zone on B.Cu, net B-
- added copper zone on B.Cu, net GND
Other:
- board outline added: 87.4 x 100.3 mm

Commit message: v1.0
Parts:
- added J1: B-, TerminalBlock_Phoenix:TerminalBlock_Phoenix_MKDS-1,5-2-5.08_1x02_P5.08mm_Horizontal, F.Cu at (242.8, 120.7)
- added J3: INPUT, TerminalBlock_4Ucon:TerminalBlock_4Ucon_1x02_P3.50mm_Horizontal, F.Cu at (190.5, 100.1)
- moved C15 31.2 mm to (215.9, 103.4)
- moved C16 26.3 mm to (219.7, 39.9)
- moved R15 3.30 mm to (200.9, 124.2)
- moved C1 1.60 mm to (189.8, 111.8)
- moved R1 1.27 mm to (195.6, 100.1)
- moved R2 1.27 mm to (203.2, 104.8)
Routing:
- net GND: track 43.5 -> 15.5 mm
- net B-: track 0.00 -> 20.5 mm
- net INPUT: track 0.00 -> 8.43 mm
- net CHASSIS: track 11.3 -> 14.7 mm
- net Net-(C1-Pad2): track 11.4 -> 14.3 mm
- net Net-(Q1-B): track 23.3 -> 25.6 mm

Commit message: Power supply
Parts:
- added ?: , , F.Cu at (243.8, 119.4)
- added ?: , , F.Cu at (243.8, 43.2)
- added PIC1: LOGO, LOGO, F.Cu at (193.5, 48.8)
- J1: value B- -> SPEAKER; footprint TerminalBlock_Phoenix:TerminalBlock_Phoenix_MKDS-1,5-2-5.08_1x02_P5.08mm_Horizontal -> TerminalBlock_Phoenix:TerminalBlock_Phoenix_MKDS-1,5-2_1x02_P5.00mm_Horizontal
- moved J1 45.9 mm to (229.5, 76.7), turned to 180 degrees
- moved R3 24.3 mm to (192.5, 70.4)
- moved R4 24.1 mm to (198.4, 70.4)
- moved Q4 18.2 mm to (195.8, 86.9)
- moved Q3 17.8 mm to (190.0, 86.9)
- moved R25 7.85 mm to (229.1, 66.8)
- moved R24 7.72 mm to (223.1, 66.8)
- moved Q2 5.79 mm to (195.8, 91.9)
- moved C3 4.57 mm to (225.3, 86.4)
- moved R26 4.57 mm to (229.1, 91.8)
- moved R27 4.57 mm to (223.1, 99.3)
- moved Q1 1.55 mm to (190.0, 91.9)
- moved D4 0.64 mm to (262.8, 103.9)
- moved D5 0.63 mm to (258.1, 96.3)
Connections:
- net INPUT renamed /INPUT
- net Net-(Q2-C) renamed /LTP COM
- J1 pad 1: B- -> /SPEAKER
- J1 pad 2: (no net) -> GND
- R21 pad 2: SPEAKER -> /SPEAKER
Routing:
- net /LTP COM: track 39.5 -> 0.00 mm
- net Net-(Q13-E): track 86.8 -> 96.9 mm
- net Net-(Q1-C): track 61.5 -> 52.7 mm
- net Net-(Q3-E): track 16.7 -> 8.89 mm
- net /SPEAKER: track 0.00 -> 7.37 mm
- net Net-(Q4-E): track 14.7 -> 8.89 mm
- net Net-(D6-A): track 99.5 -> 94.9 mm
- net Net-(Q14-B): track 21.3 -> 25.7 mm
- net Net-(Q2-B): track 24.0 -> 28.1 mm
- net Net-(Q12-E): track 68.5 -> 66.6 mm
- net Net-(Q10-E): track 81.1 -> 79.4 mm
- net Net-(D3-K): track 61.6 -> 60.2 mm
- net Net-(Q1-B): track 25.6 -> 26.9 mm
- net Net-(Q1-E): track 34.2 -> 33.5 mm
- net Net-(C3-Pad2): track 6.07 -> 6.69 mm
- added copper zone on B.Cu, net /LTP COM
- added copper zone on F.Cu, net /LTP COM
Other:
- board size 87.4 x 100.3 mm -> 87.4 x 101.9 mm
- board text added: "Designed by Pontus Rydin. https://github.com/prydin/classab-amp"

Commit message: Post 1.0 adjutments
Parts:
- added ?: , , F.Cu at (235.0, 103.1)
Other:
- board text added: "GND"
- board text added: "V+"
- board text added: "V-"
Changed lines of the file:
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@@
 		)
 	)
+	(footprint ""
+		(layer "F.Cu")
+		(at 234.966 103.124)
+		(property "Reference" ""
+			(at 0 0 0)
+			(layer "F.SilkS")
+			(effects
+				(font
+					(size 1.27 1.27)
+					(thickness 0.15)
+				)
+			)
+		)
+		(property "Value" ""
+			(at 0 0 0)
+			(layer "F.Fab")
+			(effects
+				(font
+					(size 1.27 1.27)
+					(thickness 0.15)
+				)
+			)
+		)
+		(property "Footprint" ""
+			(at 0 0 0)
+			(layer "F.Fab")
+			(hide yes)
+			(effects
+				(font
+					(size 1.27 1.27)
+					(thickness 0.15)
+				)
+			)
+		)
+		(property "Datasheet" ""
+			(at 0 0 0)
+			(layer "F.Fab")
+			(hide yes)
+			(effects
+				(font
+					(size 1.27 1.27)
+					(thickness 0.15)
+				)
+			)
+		)
+		(property "Description" ""
+			(at 0 0 0)
+			(layer "F.Fab")
+			(hide yes)
+			(effects
+				(font
+					(size 1.27 1.27)
+					(thickness 0.15)
+				)
+			)
+		)
+		(pad "1" thru_hole circle
+			(at 1 0)
+			(size 2.7 2.7)
+			(drill 1.5)
+			(layers "*.Cu" "*.Mask")
+			(remove_unused_layers no)
+			(net 25 "GND")
+		)
+	)
 	(footprint "Package_TO_SOT_THT:TO-92_Inline"
 		(layer "F.Cu")
@@
 		(tags "THT Terminal Block Phoenix MKDS-1,5-2 pitch 5mm size 10x9.8mm^2 drill 1.3mm pad 2.6mm")
 		(property "Reference" "J1"
-			(at 2.46 6.096 360)
+			(at 2.46 6.096 0)
 			(layer "F.SilkS")
 			(effects
@@
 		)
 		(property "Value" "SPEAKER"
-			(at 2.5 5.66 360)
+			(at 2.5 5.66 0)
 			(layer "F.Fab")
 			(effects
@@
 		)
 		(fp_text user "${REFERENCE}"
-			(at 2.5 3.2 360)
+			(at 2.5 3.2 0)
 			(layer "F.Fab")
 			(effects
@@
 		(layer "Edge.Cuts")
 	)
+	(gr_text "V+"
+		(at 244.348 40.386 0)
+		(layer "F.SilkS")
+		(effects
+			(font
+				(size 1 1)
+				(thickness 0.1)
+			)
+			(justify left bottom)
+		)
+	)
+	(gr_text "V-"
+		(at 244.348 123.444 0)
+		(layer "F.SilkS")
+		(effects
+			(font
+				(size 1 1)
+				(thickness 0.1)
+			)
+			(justify left bottom)
+		)
+	)
 	(gr_text "Designed by Pontus Rydin. https://github.com/prydin/classab-amp"
 		(at 194.564 131.064 0)
@@
 		)
 	)
+	(gr_text "GND"
+		(at 238.252 103.378 0)
+		(layer "F.SilkS")
+		(effects
+			(font
+				(size 1 1)
+				(thickness 0.1)
+			)
+			(justify left bottom)
+		)
+	)
 	(segment
 		(start 210.312 108.866)
@@
 		(polygon
 			(pts
-				(xy 242.058 115.167) (xy 252.218 82.147) (xy 271.141 82.147) (xy 271.141 125.962) (xy 185.8772 126.4412)
+				(xy 242.058 115.167) (xy 252.218 82.147) (xy 271.141 82.147) (xy 271.018 126.492) (xy 185.8772 126.4412)
 				(xy 185.8772 115.2652) (xy 196.596 115.316) (xy 224.913 115.167)
 			)

Commit message: Post build adjustments
Parts:
- added C6: 100n, Capacitor_THT:C_Rect_L7.2mm_W3.0mm_P5.00mm_FKS2_FKP2_MKS2_MKP2, F.Cu at (262.6, 74.7)
- added D10: 1N4004, Diode_THT:D_DO-41_SOD81_P10.16mm_Horizontal, F.Cu at (240.8, 111.3)
- added D7: 1N4004, Diode_THT:D_DO-41_SOD81_P10.16mm_Horizontal, F.Cu at (240.8, 41.9)
- added D8: 1N4004, Diode_THT:D_DO-41_SOD81_P10.16mm_Horizontal, F.Cu at (253.0, 42.9)
- added D9: 1N4004, Diode_THT:D_DO-41_SOD81_P10.16mm_Horizontal, F.Cu at (253.7, 118.1)
- C4: footprint Capacitor_THT:CP_Radial_D4.0mm_P1.50mm -> Capacitor_THT:CP_Radial_D8.0mm_P5.00mm
- R10, R14: value 1k -> 150
- R12: value 6.8k -> 15k
- R5: value 2.2k -> 1k
- moved ? 3.57 mm to (247.4, 119.4)
- moved ? 3.57 mm to (247.4, 43.2)
- moved C4 1.80 mm to (214.4, 80.0)
Routing:
- net Net-(D3-K): track 60.2 -> 68.4 mm
- net Net-(D6-A): track 94.9 -> 100.5 mm
- net Net-(Q1-C): track 52.7 -> 47.9 mm
- net Net-(C4-Pad2): track 7.35 -> 4.78 mm
- net Net-(Q2-B): track 28.1 -> 29.1 mm
- net Net-(Q7-B): track 19.2 -> 19.9 mm
- removed copper zone on F.Cu, net /LTP COM

Commit message: Added ver 2 SPICE design
Parts:
- D3, D6: value 1N4001 -> 1N4004
- R13, R6: value 47k -> 10k
- moved R12 0.89 mm to (255.9, 84.6)
- moved R14 0.89 mm to (261.4, 84.6)
Routing:
- net Net-(D3-K): track 68.4 -> 69.3 mm

Commit message: Update gerber files
Parts:
- added C7: 10n, Capacitor_THT:C_Rect_L7.2mm_W3.0mm_P5.00mm_FKS2_FKP2_MKS2_MKP2, F.Cu at (193.0, 119.9)
- added C8: 4.7n, Capacitor_THT:C_Rect_L7.2mm_W3.0mm_P5.00mm_FKS2_FKP2_MKS2_MKP2, F.Cu at (262.6, 91.4)
- R15: value 10 -> 220
- moved R14 3.81 mm to (257.6, 84.6)
- moved R12 2.41 mm to (253.5, 84.6)
- moved R13 0.90 mm to (249.4, 92.2)
Routing:
- net GND: track 15.5 -> 29.8 mm
- net Net-(D4-A): track 29.0 -> 34.0 mm
- net Net-(D3-K): track 69.3 -> 74.3 mm
- net Net-(Q8-E): track 6.40 -> 10.2 mm
- net Net-(R12-Pad1): track 8.85 -> 7.33 mm

Commit message: WIP
Parts:
- removed R8: 1k, Resistor_THT:R_Axial_DIN0204_L3.6mm_D1.6mm_P7.62mm_Horizontal
- added R22: 150, Resistor_THT:R_Axial_DIN0204_L3.6mm_D1.6mm_P7.62mm_Horizontal, F.Cu at (191.0, 94.7)
- added R23: 150, Resistor_THT:R_Axial_DIN0204_L3.6mm_D1.6mm_P7.62mm_Horizontal, F.Cu at (197.1, 94.7)
- moved Q1 12.2 mm to (190.0, 79.8)
- moved Q2 12.2 mm to (195.8, 79.8)
- moved Q3 12.2 mm to (190.0, 74.7)
- moved Q4 12.2 mm to (195.8, 74.7)
- moved R4 9.66 mm to (198.6, 60.7)
- moved R3 9.65 mm to (192.5, 60.7)
- moved C2 4.16 mm to (204.7, 97.0), turned to 90 degrees
- moved R7 4.15 mm to (204.2, 80.5)
- moved C12 2.80 mm to (212.7, 93.6)
- moved Q14 1.91 mm to (218.9, 91.9)
Connections:
- C5 pad 1: Net-(Q6-B) -> Net-(Q1-C)
- Q2 pad 3: Net-(Q1-E) -> Net-(Q2-E)
- Q5 pad 1: Net-(Q1-E) -> Net-(Q5-C)
- Q6 pad 3: Net-(Q6-B) -> Net-(Q1-C)
Routing:
- net Net-(Q5-C): track 0.00 -> 32.0 mm
- net Net-(Q1-E): track 33.5 -> 7.25 mm
- net Net-(Q1-B): track 26.9 -> 40.6 mm
- net Net-(Q6-B): track 11.7 -> 0.00 mm
- net Net-(Q2-E): track 0.00 -> 7.14 mm
- net Net-(C4-Pad2): track 4.78 -> 9.25 mm
- net Net-(Q3-E): track 8.89 -> 6.35 mm
- net Net-(Q4-E): track 8.89 -> 6.45 mm
- net Net-(Q2-B): track 29.1 -> 26.8 mm
- net Net-(D6-K): track 67.4 -> 65.5 mm
- net Net-(D3-A): track 41.7 -> 40.4 mm
- net Net-(Q13-E): track 96.9 -> 95.7 mm
- net Net-(Q14-B): track 25.7 -> 24.7 mm
- net Net-(Q1-C): track 47.9 -> 47.6 mm, vias 0 -> 2
