File: kicad/power_supply/power_supply.kicad_sch (KiCad schematic)
At the start: 8 parts

Commit message: Power supply
Parts:
- removed D1, D2, D3, D4: 1N5400, Diode_THT:D_DO-201AD_P15.24mm_Horizontal, symbol Diode:1N5400
- added D1, D2, D3, D4: GI754, Diode_THT:D_P600_R-6_P12.70mm_Horizontal, symbol Device:D
- added J1: AC IN, TerminalBlock_Phoenix:TerminalBlock_Phoenix_PT-1,5-3-3.5-H_1x03_P3.50mm_Horizontal, symbol Connector:Screw_Terminal_01x03
- added J2: DC OUT, TerminalBlock_Phoenix:TerminalBlock_Phoenix_PT-1,5-3-3.5-H_1x03_P3.50mm_Horizontal, symbol Connector:Screw_Terminal_01x03
- C3, C4: footprint (none) -> Capacitor_THT:C_Rect_L7.2mm_W5.5mm_P5.00mm_FKS2_FKP2_MKS2_MKP2
Connections:
- net GND: now also J1.2 (Pin_2), J2.2 (Pin_2)
- net B+: no longer names the net of C1.1, C3.1
- net B+: now also D1.1 (K), D3.1 (K), J2.3 (Pin_3)
- net B-: no longer names the net of C2.2, C4.2
- net B-: now also D2.2 (A), D4.2 (A), J2.1 (Pin_1)
- new net: D2.1 (K), D3.2 (A), J1.1 (Pin_1)
- new net: D1.2 (A), D4.1 (K), J1.3 (Pin_3)

Commit message: Added images
Connections:
- net V+: now reaches C1.1, C3.1, D1.1 (K), D3.1 (K), J2.3 (Pin_3)
- net AC2: now reaches D2.1 (K), D3.2 (A), J1.1 (Pin_1)
- net V-: now reaches C2.2, C4.2, D2.2 (A), D4.2 (A), J2.1 (Pin_1)
- net AC1: now reaches D1.2 (A), D4.1 (K), J1.3 (Pin_3)
Other:
- moved on the sheet: J1
Changed lines of the file:
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@@
 	(wire
 		(pts
-			(xy 68.58 119.38) (xy 85.09 119.38)
+			(xy 67.31 119.38) (xy 85.09 119.38)
 		)
 		(stroke
@@
 	(wire
 		(pts
-			(xy 66.04 118.11) (xy 68.58 118.11)
+			(xy 64.77 118.11) (xy 67.31 118.11)
 		)
 		(stroke
@@
 	(wire
 		(pts
-			(xy 66.04 123.19) (xy 68.58 123.19)
+			(xy 64.77 123.19) (xy 67.31 123.19)
 		)
 		(stroke
@@
 	(wire
 		(pts
-			(xy 68.58 121.92) (xy 68.58 123.19)
+			(xy 67.31 121.92) (xy 67.31 123.19)
 		)
 		(stroke
@@
 	(wire
 		(pts
-			(xy 66.04 120.65) (xy 99.06 120.65)
+			(xy 64.77 120.65) (xy 99.06 120.65)
 		)
 		(stroke
@@
 	(wire
 		(pts
-			(xy 68.58 121.92) (xy 72.39 121.92)
+			(xy 67.31 121.92) (xy 72.39 121.92)
 		)
 		(stroke
@@
 	(wire
 		(pts
-			(xy 68.58 118.11) (xy 68.58 119.38)
+			(xy 67.31 118.11) (xy 67.31 119.38)
 		)
 		(stroke
@@
 			(width 0)
 			(type default)
+		)
+	)
+	(label "AC1"
+		(at 67.31 118.11 0)
+		(fields_autoplaced yes)
+		(effects
+			(font
+				(size 1.27 1.27)
+			)
+			(justify left bottom)
+		)
+	)
+	(label "AC2"
+		(at 67.31 123.19 0)
+		(fields_autoplaced yes)
+		(effects
+			(font
+				(size 1.27 1.27)
+			)
+			(justify left bottom)
+		)
+	)
+	(label "V-"
+		(at 132.08 135.89 0)
+		(fields_autoplaced yes)
+		(effects
+			(font
+				(size 1.27 1.27)
+			)
+			(justify left bottom)
+		)
+	)
+	(label "V+"
+		(at 132.08 106.68 0)
+		(fields_autoplaced yes)
+		(effects
+			(font
+				(size 1.27 1.27)
+			)
+			(justify left bottom)
 		)
 	)
@@
 	(symbol
 		(lib_id "Connector:Screw_Terminal_01x03")
-		(at 60.96 120.65 180)
+		(at 59.69 120.65 180)
 		(unit 1)
 		(exclude_from_sim no)
@@
 		(fields_autoplaced yes)
 		(property "Reference" "J1"
-			(at 60.96 111.76 0)
+			(at 59.69 111.76 0)
 			(effects
 				(font
@@
 		)
 		(property "Value" "AC IN"
-			(at 60.96 114.3 0)
+			(at 59.69 114.3 0)
 			(effects
 				(font
@@
 		)
 		(property "Footprint" "TerminalBlock_Phoenix:TerminalBlock_Phoenix_PT-1,5-3-3.5-H_1x03_P3.50mm_Horizontal"
-			(at 60.96 120.65 0)
+			(at 59.69 120.65 0)
 			(effects
 				(font
@@
 		)
 		(property "Datasheet" "~"
-			(at 60.96 120.65 0)
+			(at 59.69 120.65 0)
 			(effects
 				(font
@@
 		)
 		(property "Description" "Generic screw terminal, single row, 01x03, script generated (kicad-library-utils/schlib/autogen/connector/)"
-			(at 60.96 120.65 0)
-			(effects
-				(font
+			(at 59.69 120.65 0)
+			(effects
+				(font

Commit message: Added ver 2 SPICE design
Parts:
- added C5, C6: 4700u, Capacitor_THT:CP_Radial_D18.0mm_P7.50mm, symbol Device:C_Polarized
Connections:
- net GND: now also C5.2, C6.1
- net V+: now also C5.1
- net V-: now also C6.2
Other:
- moved on the sheet: C3, C4, J2

Commit message: WIP
Parts:
- added R1, R2: 1k, Resistor_THT:R_Axial_DIN0414_L11.9mm_D4.5mm_P15.24mm_Horizontal, symbol Device:R
Connections:
- net GND: now also R1.2, R2.1
- net V+: now also R1.1
- net V-: now also R2.2
Other:
- note added: "5W"
- moved on the sheet: C1, C3, C5, D1, D3, J2
